File: buck-converter-high-voltage.kicad_pcb (KiCad board)
At the start: 2 copper layers, 28.5 x 21 mm, 21 parts, among them J1 Input, J2 Output, U1 MAX17574

Commit message: Change inductor value to 47µH
Parts:
- added D1: SMAJ51A, Diode_SMD:D_SMA, B.Cu at (124.6, 101.0)
- L1: value XGL6060-333 -> XGL6060-473
Routing:
- net GND: track 26.4 -> 31.4 mm
- net Vdrive: track 8.53 -> 12.9 mm
Changed lines of the file:
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@@
       (plot_on_all_layers_selection 0x0000000_00000000)
       (disableapertmacros false)
-      (usegerberextensions false)
+      (usegerberextensions true)
       (usegerberattributes true)
       (usegerberadvancedattributes true)
-      (creategerberjobfile true)
+      (creategerberjobfile false)
       (dashed_line_dash_ratio 12.000000)
       (dashed_line_gap_ratio 3.000000)
@@
       (plotinvisibletext false)
       (sketchpadsonfab false)
-      (subtractmaskfromsilk false)
+      (subtractmaskfromsilk true)
       (outputformat 1)
       (mirror false)
-      (drillshape 1)
+      (drillshape 0)
       (scaleselection 1)
-      (outputdirectory "")
+      (outputdirectory "gerber")
     )
   )
@@
   (net 16 "unconnected-(U1-NC-Pad13)")
   (net 17 "unconnected-(U1-~{RESET}-Pad14)")
-  (net 18 "Net-(U1-EXTVCC)")
+  (net 18 "Net-(#FLG04-pwr)")
   (footprint "Resistor_SMD:R_0603_1608Metric" (layer "F.Cu")
     (at 135.95 106.8 -90)
@@
         (effects (font (size 1 1) (thickness 0.15)))
     )
-    (fp_text user "VCC" (at 2.525 5.275 270 unlocked) (layer "B.SilkS")
+    (fp_text user "VCC" (at 2.575 4.575 unlocked) (layer "B.SilkS")
         (effects (font (size 0.8 0.8) (thickness 0.1)) (justify mirror))
     )
@@
         (effects (font (size 0.8 0.8) (thickness 0.1)) (justify mirror))
     )
-    (fp_text user "GND" (at 0.025 5.275 270 unlocked) (layer "B.SilkS")
+    (fp_text user "GND" (at -3.025 2.575 unlocked) (layer "B.SilkS")
         (effects (font (size 0.8 0.8) (thickness 0.1)) (justify mirror))
     )
@@
       (net 13 "Net-(U1-RT)") (pinfunction "RT") (pintype "input"))
     (pad "20" smd roundrect (at 1 -2.45 270) (size 0.25 0.85) (layers "F.Cu" "F.Paste" "F.Mask") (roundrect_rratio 0.25)
-      (net 18 "Net-(U1-EXTVCC)") (pinfunction "EXTVCC") (pintype "power_in"))
+      (net 18 "Net-(#FLG04-pwr)") (pinfunction "EXTVCC") (pintype "power_in"))
     (pad "21" smd roundrect (at 0.5 -2.45 270) (size 0.25 0.85) (layers "F.Cu" "F.Paste" "F.Mask") (roundrect_rratio 0.25)
       (net 2 "GND") (pinfunction "SGND") (pintype "power_in"))
@@
       (net 2 "GND") (pintype "passive"))
     (pad "2" smd roundrect (at 0.775 0) (size 0.9 0.95) (layers "F.Cu" "F.Paste" "F.Mask") (roundrect_rratio 0.25)
-      (net 18 "Net-(U1-EXTVCC)") (pintype "passive"))
+      (net 18 "Net-(#FLG04-pwr)") (pintype "passive"))
     (model "${KICAD6_3DMODEL_DIR}/Capacitor_SMD.3dshapes/C_0603_1608Metric.wrl"
       (offset (xyz 0 0 0))
@@
       (stroke (width 0.1) (type solid)) (layer "F.Fab"))
     (pad "1" smd roundrect (at -0.825 0 270) (size 0.8 0.95) (layers "F.Cu" "F.Paste" "F.Mask") (roundrect_rratio 0.25)
-      (net 18 "Net-(U1-EXTVCC)") (pintype "passive"))
+      (net 18 "Net-(#FLG04-pwr)") (pintype "passive"))
     (pad "2" smd roundrect (at 0.825 0 270) (size 0.8 0.95) (layers "F.Cu" "F.Paste" "F.Mask") (roundrect_rratio 0.25)
       (net 8 "+6V") (pintype "passive"))
@@
         (effects (font (size 0.8 0.8) (thickness 0.1)))
     )
-    (fp_text value "XGL6060-333" (at 0 4.38 90) (layer "F.Fab")
+    (fp_text value "XGL6060-473" (at 0 4.38 90) (layer "F.Fab")
         (effects (font (size 1 1) (thickness 0.15)))
     )
@@
       (net 5 "Net-(U1-FB)") (pintype "passive"))
     (model "${KICAD6_3DMODEL_DIR}/Resistor_SMD.3dshapes/R_0603_1608Metric.wrl"
+      (offset (xyz 0 0 0))
+      (scale (xyz 1 1 1))
+      (rotate (xyz 0 0 0))
+    )
+  )
+  (footprint "Diode_SMD:D_SMA" (layer "B.Cu")
+    (at 124.6 101)
+    (descr "Diode SMA (DO-214AC)")
+    (tags "Diode SMA (DO-214AC)")
+    (property "Sheetfile" "buck-converter-high-voltage.kicad_sch")
+    (property "Sheetname" "")
+    (property "ki_description" "Zener diode")
+    (property "ki_keywords" "diode")
+    (attr smd)
+    (fp_text reference "D1" (at 0 -2.2) (layer "B.SilkS")
+        (effects (font (size 0.8 0.8) (thickness 0.1)) (justify mirror))
+    )
+    (fp_text value "SMAJ51A" (at 0 -2.6) (layer "B.Fab")
+        (effects (font (size 1 1) (thickness 0.15)) (justify mirror))
+    )
+    (fp_text user "${REFERENCE}" (at 0 2.5) (layer "B.Fab")
+        (effects (font (size 1 1) (thickness 0.15)) (justify mirror))
+    )
+    (fp_line (start -3.51 -1.65) (end 2 -1.65)
+      (stroke (width 0.12) (type solid)) (layer "B.SilkS"))
+    (fp_line (start -3.51 1.65) (end -3.51 -1.65)
+      (stroke (width 0.12) (type solid)) (layer "B.SilkS"))
+    (fp_line (start -3.51 1.65) (end 2 1.65)
+      (stroke (width 0.12) (type solid)) (layer "B.SilkS"))
+    (fp_line (start -3.5 -1.75) (end -3.5 1.75)
+      (stroke (width 0.05) (type solid)) (layer "B.CrtYd"))
+    (fp_line (start -3.5 1.75) (end 3.5 1.75)
+      (stroke (width 0.05) (type solid)) (layer "B.CrtYd"))
+    (fp_line (start 3.5 -1.75) (end -3.5 -1.75)
+      (stroke (width 0.05) (type solid)) (layer "B.CrtYd"))
+    (fp_line (start 3.5 1.75) (end 3.5 -1.75)
+      (stroke (width 0.05) (type solid)) (layer "B.CrtYd"))
+    (fp_line (start -2.3 -1.5) (end -2.3 1.5)
+      (stroke (width 0.1) (type solid)) (layer "B.Fab"))
+    (fp_line (start -0.64944 -0.00102) (end -1.55114 -0.00102)
+      (stroke (width 0.1) (type solid)) (layer "B.Fab"))
+    (fp_line (start -0.64944 -0.00102) (end 0.50118 -0.75032)
+      (stroke (width 0.1) (type solid)) (layer "B.Fab"))
+    (fp_line (start -0.64944 -0.00102) (end 0.50118 0.79908)
+      (stroke (width 0.1) (type solid)) (layer "B.Fab"))
+    (fp_line (start -0.64944 0.79908) (end -0.64944 -0.80112)
+      (stroke (width 0.1) (type solid)) (layer "B.Fab"))
+    (fp_line (start 0.50118 -0.75032) (end 0.50118 0.79908)
+      (stroke (width 0.1) (type solid)) (layer "B.Fab"))
+    (fp_line (start 0.50118 -0.00102) (end 1.4994 -0.00102)
+      (stroke (width 0.1) (type solid)) (layer "B.Fab"))
+    (fp_line (start 2.3 -1.5) (end -2.3 -1.5)
+      (stroke (width 0.1) (type solid)) (layer "B.Fab"))
+    (fp_line (start 2.3 1.5) (end -2.3 1.5)
+      (stroke (width 0.1) (type solid)) (layer "B.Fab"))
+    (fp_line (start 2.3 1.5) (end 2.3 -1.5)
+      (stroke (width 0.1) (type solid)) (layer "B.Fab"))
+    (pad "1" smd roundrect (at -2 0) (size 2.5 1.8) (layers "B.Cu" "B.Paste" "B.Mask") (roundrect_rratio 0.1388888889)
+      (net 9 "Vdrive") (pinfunction "K") (pintype "passive"))
+    (pad "2" smd roundrect (at 2 0) (size 2.5 1.8) (layers "B.Cu" "B.Paste" "B.Mask") (roundrect_rratio 0.1388888889)
+      (net 2 "GND") (pinfunction "A") (pintype "passive"))
+    (model "${KICAD6_3DMODEL_DIR}/Diode_SMD.3dshapes/D_SMA.wrl"
       (offset (xyz 0 0 0))
       (scale (xyz 1 1 1))
@@
   (via (at 126.5 108) (size 0.7) (drill 0.3) (layers "F.Cu" "B.Cu") (free) (net 2))
   (via (at 135 95.75) (size 0.7) (drill 0.3) (layers "F.Cu" "B.Cu") (free) (net 2))
+  (segment (start 124.775 102.825) (end 126.6 101) (width 1) (layer "B.Cu") (net 2))
+  (segment (start 124.775 105.235) (end 124.775 102.825) (width 1) (layer "B.Cu") (net 2))
   (segment (start 133.95 104.8) (end 134.25 104.5) (width 0.25) (layer "F.Cu") (net 3))
   (segment (start 131.45 106.025) (end 132.675 104.8) (width 0.25) (layer "F.Cu") (net 3))
@@
   (segment (start 138.925 101.55) (end 138.95 101.575) (width 0.25) (layer "F.Cu") (net 7))
   (segment (start 136.7 101.55) (end 138.925 101.55) (width 0.25) (layer "F.Cu") (net 7))
-  (segment (start 141.5 104.5) (end 138.95 107.05) (width 0.25) (layer "F.Cu") (net 8))
-  (segment (start 142.75 102.25) (end 141.5 103.5) (width 0.25) (layer "F.Cu") (net 8))
-  (segment (start 148 98.5) (end 148 101.5) (width 0.25) (layer "F.Cu") (net 8))
-  (segment (start 141.5 103.5) (end 141.5 104.5) (width 0.25) (layer "F.Cu") (net 8))
+  (segment (start 141.4 104.625) (end 138.95 107.075) (width 0.25) (layer "F.Cu") (net 8))
+  (segment (start 148 98.5) (end 148 101.8) (width 0.25) (layer "F.Cu") (net 8))
+  (segment (start 148 101.8) (end 145.175 104.625) (width 0.25) (layer "F.Cu") (net 8))
+  (segment (start 146.23 96.73) (end 148 98.5) (width 0.25) (layer "F.Cu") (net 8))
   (segment (start 144 96.73) (end 146.23 96.73) (width 0.25) (layer "F.Cu") (net 8))
-  (segment (start 146.23 96.73) (end 148 98.5) (width 0.25) (layer "F.Cu") (net 8))
   (segment (start 138.95 107.55) (end 138.95 107.075) (width 0.25) (layer "F.Cu") (net 8))
-  (segment (start 138.95 107.05) (end 138.95 107.075) (width 0.25) (layer "F.Cu") (net 8))
-  (segment (start 148 101.5) (end 147.25 102.25) (width 0.25) (layer "F.Cu") (net 8))
-  (segment (start 147.25 102.25) (end 142.75 102.25) (width 0.25) (layer "F.Cu") (net 8))
+  (segment (start 145.175 104.625) (end 141.4 104.625) (width 0.25) (layer "F.Cu") (net 8))
   (segment (start 135.375 108.55) (end 137.95 108.55) (width 0.25) (layer "F.Cu") (net 8))
   (segment (start 134.45 107.625) (end 135.375 108.55) (width 0.25) (layer "F.Cu") (net 8))
@@
   (segment (start 122.235 105.235) (end 122.235 103.265) (width 0.25) (layer "F.Cu") (net 9))
   (segment (start 122.25 103.25) (end 122.235 103.265) (width 0.25) (layer "F.Cu") (net 9))
+  (segment (start 122.235 105.235) (end 122.235 101.365) (width 1) (layer "B.Cu") (net 9))
+  (segment (start 122.235 101.365) (end 122.6 101) (width 1) (layer "B.Cu") (net 9))
   (segment (start 123.5 103.5) (end 126 101) (width 0.25) (layer "F.Cu") (net 10))
   (segment (start 124.775 107.775) (end 123.5 106.5) (width 0.25) (layer "F.Cu") (net 10))
@@
         (xy 148.2 98.8)
         (xy 140.2 98.8)
-        (xy 140.2 98.8)
         (xy 135.45 98.8)
